File: STM32_sheild/STM32_sheild.kicad_sch (KiCad schematic)
At the start: 5 parts, among them J1 CN7, J2 CN10

Commit message: changes to shield schematic
Parts:
- added P1: USB_C_Plug_USB2.0, symbol Connector:USB_C_Plug_USB2.0
- added U1: MCP73831-2-MC, Package_DFN_QFN:DFN-8-1EP_3x2mm_P0.5mm_EP1.7x1.4mm, symbol Battery_Management:MCP73831-2-MC
- added U2: OPA333xxDBV, Package_TO_SOT_SMD:SOT-23-5, symbol Amplifier_Operational:OPA333xxDBV
- added U3: TPS63030DSK, Package_SON:WSON-10-1EP_2.5x2.5mm_P0.5mm_EP1.2x2mm, symbol Regulator_Switching:TPS63030DSK
Connections:
- new net: P1.A1 (GND), P1.A12 (GND), P1.B1 (GND), P1.B12 (GND)
- new net: P1.A4 (VBUS), P1.A9 (VBUS), P1.B4 (VBUS), P1.B9 (VBUS)
- new net: U3.11 (PGND), U3.3 (PGND)
- new net: U1.1 (V_{DD}), U1.2 (V_{DD})
- new net: U1.3 (V_{BAT}), U1.4 (V_{BAT})

Commit message: Placing first components on schematic
Parts:
- removed P1: USB_C_Plug_USB2.0, symbol Connector:USB_C_Plug_USB2.0
- removed U3: TPS63030DSK, Package_SON:WSON-10-1EP_2.5x2.5mm_P0.5mm_EP1.2x2mm, symbol Regulator_Switching:TPS63030DSK
- added B1: 1042P, 18650_cradle:1042P_KEY, symbol 2026-07-04_16-48-10:1042P
- added C1, C2: 10uF, Capacitor_SMD:C_0805_2012Metric, symbol Device:C
- added C3: 100n, Capacitor_SMD:C_0805_2012Metric, symbol Device:C
- added D1: ESD9B3.3ST5G, Diode_SMD:D_SOD-923, symbol Diode:ESD9B3.3ST5G
- added J3: 61612002121503, KiCad_SMB_coax:61612002121503, symbol 61612002121503:61612002121503
- added J4: 632722100213, KiCad_wurth_USB-C_PD_connector:632722100213, symbol 632722100213:632722100213
- added JP1: Jumper_3_Bridged12, Jumper:SolderJumper-3_P1.3mm_Bridged2Bar12_Pad1.0x1.5mm, symbol Jumper:Jumper_3_Bridged12
- added R1: 10k, Resistor_SMD:R_0805_2012Metric, symbol Device:R
- added R2: 330k, Resistor_SMD:R_0805_2012Metric, symbol Device:R
- added R3: 2.2k, Resistor_SMD:R_0805_2012Metric, symbol Device:R
- added R4: 10R, Resistor_SMD:R_0805_2012Metric, symbol Device:R
- added R5: 100R, Resistor_SMD:R_0805_2012Metric, symbol Device:R
- added U4: TPS63031DSK, Package_SON:WSON-10-1EP_2.5x2.5mm_P0.5mm_EP1.2x2mm, symbol Regulator_Switching:TPS63031DSK
Connections:
- net GNDA is gone; now on net GND: J2.32 (Pin_32)
- net GND: now also U2.2 (V-), C1.2, C2.2, C3.2, D1.2 (A2), J3.2, J3.3, J3.4, J3.5, R1.2
- net VDD: now also R4.2
- net ADC1: now reaches J1.28 (Pin_28)
- net ADC1: now also C1.1, R3.2
- net ADC2: now reaches J1.30 (Pin_30)
- net at U2.1: now also R2.2, R3.1
- net at U2.3 (+): now also D1.1 (A1), R5.2
- net at U2.4 (-): now also R1.1, R2.1
- net at U2.5 (V+): now also C2.1, C3.1, R4.1
- new net: U4.11 (PGND), U4.3 (PGND)
- new net: J3.1, R5.1
Other:
- moved on the sheet: J1, J2, U1, U2

Commit message: more changes to schematic mainly
Parts:
- added C4, C5: 4.7uF, Capacitor_SMD:C_0805_2012Metric, symbol Device:C
- added C6: 100n, Capacitor_SMD:C_0805_2012Metric, symbol Device:C
- added C7, C8, C9: 10uF, Capacitor_SMD:C_0805_2012Metric, symbol Device:C
- added L1: L, symbol Device:L
- added L2: LPS3015-152MRC, LPS3015-152MRC:IND_LPS3015-152MRC, symbol LPS3015-152MRC:LPS3015-152MRC
- added R6, R7: 5.1k, Resistor_SMD:R_0805_2012Metric, symbol Device:R
- added R8: 2k, Resistor_SMD:R_0805_2012Metric, symbol Device:R
Connections:
- net +BATT: now also B1.2, U1.3 (V_{BAT}), U1.4 (V_{BAT}), U4.5 (VIN), C5.1, C7.1; no longer J1.33 (Pin_33)
- net GND: now also B1.1, J4.A12 (GROUND_1), J4.B12 (GROUND_2), U1.6 (V_{SS}), U4.11 (PGND), U4.3 (PGND), U4.9 (GND), C4.2, C5.2, C6.2, C7.2, C8.2, C9.2, R6.2, R7.2, R8.2
- net at J4.A5 (CC1): now also R7.1
- net V_USB: now reaches J4.A9 (VBUS_1)
- net V_USB: now also J4.B9 (VBUS_2), U1.1 (V_{DD}), U1.2 (V_{DD}), C4.1
- net at J4.B5 (CC2): now also R6.1
- net +3.3V: now reaches U4.1 (VOUT)
- net +3.3V: now also U4.10 (FB), C8.1, C9.1
- net at U4.2 (L2): now also L1.1
- net at U4.4 (L1): now also L1.2
- net at U4.6 (EN): now also U4.7 (PS/SYNC), U4.8 (VINA), C6.1
- net at U1.5 (STAT): now also R8.1
Other:
- moved on the sheet: B1, J4, U1, U4

Commit message: more changes to schematic and layout
Parts:
- removed L1: L, symbol Device:L
- added D2: LED, LED_SMD:LED_0805_2012Metric, symbol Device:LED
- added R9: 470R, Resistor_SMD:R_0805_2012Metric, symbol Device:R
- renumbered L2 to L1
Connections:
- net +3.3V: now also JP1.3 (B); no longer C8.1, C9.1, U4.1 (VOUT), U4.10 (FB)
- net GND: now also J4.MH1, J4.MH2, J4.MH3, J4.MH4
- net VDD: now also JP1.1 (A); no longer R4.2
- net V_USB: now also D2.2 (A)
- net at R8.1: now also U1.8 (PROG); no longer U1.5 (STAT)
- net at U4.2 (L2): now also L1.1
- net at U4.4 (L1): now also L1.2
- net at JP1.2 (C): now also R4.2
- new net: R9.1, U1.5 (STAT)
- new net: D2.1 (K), R9.2
- new net +3.3V_REG: C8.1, C9.1, U4.1 (VOUT), U4.10 (FB)
Other:
- moved on the sheet: B1, C1, C2, C3, C5, C6, C7, C8, C9, D1, J1, J2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

Commit message: Starting layout routing
Parts:
- added D3: LED, LED_SMD:LED_0805_2012Metric, symbol Device:LED
- added J5: 691210910002, KiCad_wurth_2-pin_screw_terminal:691210910002, symbol 691210910002:691210910002
- added R7: 470R, Resistor_SMD:R_0805_2012Metric, symbol Device:R
- renumbered C3 to C1, C1 to C3, C7 to C5, C8 to C6, C9 to C7, C6 to C8, C5 to C9, J3 to J1, J1 to J2, J2 to J3, R4 to R1, R8 to R10, R5 to R2, R2 to R4, R1 to R5, R9 to R6, R7 to R8, R6 to R9, U2 to U1, U4 to U2, U1 to U3
Connections:
- net +3.3V_REG: now also D3.2 (A)
- net GND: now also J3.9 (Pin_9), R7.1
- net VDDA: now also J3.7 (Pin_7)
- net OPA_IN+: now reaches D1.1 (A1), R2.2, U1.3 (+)
- net OPA_out: now reaches R3.1, R4.2, U1.1
- net OPA_IN-: now reaches R4.1, R5.1, U1.4 (-)
- net OPA_VDD: now reaches C1.1, C2.1, R1.1, U1.5 (V+)
- new net: D3.1 (K), R7.2
Other:
- moved on the sheet: C6, C7

Commit message: More changes to layout, also added another opamp
Parts:
- added C10: 100n, Capacitor_SMD:C_0805_2012Metric, symbol Device:C
- added C11, C12: 10uF, Capacitor_SMD:C_0805_2012Metric, symbol Device:C
- added D4: ESD9B3.3ST5G, Diode_SMD:D_SOD-923, symbol Diode:ESD9B3.3ST5G
- added J6: 691210910002, KiCad_wurth_2-pin_screw_terminal:691210910002, symbol 691210910002:691210910002
- added JP2: Jumper_3_Bridged12, Jumper:SolderJumper-3_P1.3mm_Bridged2Bar12_Pad1.0x1.5mm, symbol Jumper:Jumper_3_Bridged12
- added R11: 100R, Resistor_SMD:R_0805_2012Metric, symbol Device:R
- added R12: 10k, Resistor_SMD:R_0805_2012Metric, symbol Device:R
- added R13: 330k, Resistor_SMD:R_0805_2012Metric, symbol Device:R
- added R14: 2.2k, Resistor_SMD:R_0805_2012Metric, symbol Device:R
- added R15: 10R, Resistor_SMD:R_0805_2012Metric, symbol Device:R
- added TP1, TP2, TP3: TestPoint, symbol Connector:TestPoint
- added U4: OPA333xxDBV, Package_TO_SOT_SMD:SOT-23-5, symbol Amplifier_Operational:OPA333xxDBV
Connections:
- net +3.3V: now also JP2.3 (B), TP2.1
- net +3.3V_REG: now also J6.1
- net ADC2: now also C12.1, R14.2
- net GND: now also D1.1 (A1), J5.2, C10.2, C11.2, C12.2, D4.2 (A2), J6.2, R12.2, TP1.1, U4.2 (V-); no longer D1.2 (A2)
- net OPA_IN+: now also D1.2 (A2), D4.1 (A1), R11.2, U4.3 (+); no longer D1.1 (A1)
- net OPA_IN-: now also R12.1, R13.1, U4.4 (-)
- net OPA_VDD: now also C10.1, C11.1, R15.1, U4.5 (V+)
- net OPA_out: now also R13.2, R14.1, U4.1
- net VDD: now also JP2.1 (A)
- net V_USB: now also TP3.1
- net at J5.1: now also R11.1
- net Coax_in: now reaches J1.1, R2.1
- new net: JP2.2 (C), R15.2
Other:
- moved on the sheet: B1, C1, C2, C3, C4, C5, C6, C7, C8, C9, D1, D2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
