File: STM32_sheild/STM32_sheild.kicad_sch (KiCad schematic)
At the start: 54 parts, among them J1 691210910002, J2 61612002121503, J3 691210910002, J4 629722010114, J5 CN10, J6 CN7, U1 DM-OLED096-636, U2 OPA333xxDBV, U3 OPA333xxDBV, U4 TPS63031DSK, U5 MCP73831-2-MC

Commit message: cleaning up drc messages
Parts:
- J4: footprint Connector_SMD_Wurth:J_Wurth_WR-USB_629722010114 -> Connector_SMD_Wurth:J_Wurth_WR-USB_629722050114
- renumbered TP5 to TP_VDD1
Changed lines of the file:
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@@
 		(dnp no)
 		(fields_autoplaced yes)
-		(property "Reference" "TP5"
+		(property "Reference" "TP_VDD1"
 			(at 237.49 36.0679 0)
 			(show_name no)
@@
 			(project "STM32_sheild"
 				(path "/da5a1e6a-2605-436b-a30c-1027586d5c0a"
-					(reference "TP5")
+					(reference "TP_VDD1")
 					(unit 1)
 				)
@@
 			)
 		)
-		(property "Footprint" "Connector_SMD_Wurth:J_Wurth_WR-USB_629722010114"
+		(property "Footprint" "Connector_SMD_Wurth:J_Wurth_WR-USB_629722050114"
 			(at 83.82 186.69 0)
 			(hide yes)
