File: STM32_sheild/STM32_sheild.kicad_pcb (KiCad board)
At the start: 2 copper layers, 99 x 83.5 mm, 54 parts, among them J1 691210910002, J2 61612002121503, J3 691210910002, J4 629722010114, J5 CN10, J6 CN7, U1 DM-OLED096-636, U2 OPA333xxDBV, U3 OPA333xxDBV, U4 TPS63031DSK, U5 MCP73831-2-MC

Commit message: cleaning up drc messages
Parts:
- J4: footprint Connector_SMD_Wurth:J_Wurth_WR-USB_629722010114 -> Connector_SMD_Wurth:J_Wurth_WR-USB_629722050114
- moved TP_VDD1 56.8 mm to (89.2, 107.8)
- moved TP_3.3V_reg1 15.5 mm to (146.2, 74.2)
- moved U1 2.31 mm to (88.1, 73.6), turned to -90 degrees
- moved J3 1.76 mm to (151.0, 73.2)
- moved R13 0.71 mm to (147.5, 97.5)
- renumbered TP5 to TP_VDD1
Routing:
- net VDD: track 8.36 -> 58.3 mm
- net VDD_STM: track 100.1 -> 70.4 mm
- net /SDA: track 39.6 -> 12.9 mm
- net GND: track 86.8 -> 104.6 mm, vias 33 -> 34
- net +3.3V_REG: track 69.2 -> 75.2 mm
- net /SCL: track 88.0 -> 84.9 mm
- net +BATT: track 59.1 -> 60.9 mm
- net V_USB: track 27.5 -> 28.3 mm
- net Net-(U5-PROG): track 2.38 -> 3.09 mm
Other:
- board text added: "3.3V buck-boost converter"
- board text added: "Charger System"
- board text added: "Sensor 1 system"
- board text added: "Sensor 2 system"
- board text removed: "Charger indicator"
