File: STM32_sheild/_restore_backup_2026-07-19T20-16-48-722/STM32_sheild.kicad_pcb (KiCad board)
At the start: 2 copper layers, 87 x 83.5 mm, 53 parts, among them J1 691210910002, J2 61612002121503, J3 691210910002, J5 CN10, J6 CN7, U1 DM-OLED096-636, U2 OPA333xxDBV, U3 OPA333xxDBV, U4 TPS63031DSK, U5 MCP73831-2-MC

Commit message: added footprint for oled + some other changes
Parts:
- removed the R14 at (90.4, 86.9)
- removed the R15 at (90.4, 89.9)
- removed TP5: TP_VDD, TestPoint:TestPoint_Keystone_5010-5014_Multipurpose
- removed TP_3.3V_reg1: TP_3.3V_reg, TestPoint:TestPoint_Keystone_5010-5014_Multipurpose
- removed TP_ADC1: TP_ADC1, TestPoint:TestPoint_Keystone_5010-5014_Multipurpose
- removed TP_ADC2: TP_ADC2, TestPoint:TestPoint_Keystone_5010-5014_Multipurpose
- removed TP_GND1: TP_GND, TestPoint:TestPoint_Keystone_5010-5014_Multipurpose
- removed TP_V_USB1: TP_V_USB, TestPoint:TestPoint_Keystone_5010-5014_Multipurpose
- removed the U1 at (86.8, 71.7)
- added J4: Conn_01x04_Pin, Connector:FanPinHeader_1x04_P2.54mm_Vertical, F.Cu at (120.5, 108.3)
- added J7: 629722010114, Connector_SMD_Wurth:J_Wurth_WR-USB_629722010114, F.Cu at (156.6, 103.8)
- added JP2: Jumper_3_Bridged12, Jumper:SolderJumper-3_P1.3mm_Bridged2Bar12_Pad1.0x1.5mm, F.Cu at (129.0, 72.5)
- added R8: 5.1k, Resistor_SMD:R_0805_2012Metric, F.Cu at (149.0, 102.0)
- added R9: 5.1k, Resistor_SMD:R_0805_2012Metric, F.Cu at (149.0, 106.0)
- moved JP1 22.7 mm to (112.5, 72.3), turned to 90 degrees
- renumbered C5 to C1, C8 to C10, C7 to C11, C4 to C2, C9 to C3, C11 to C4, C6 to C5, C1 to C6, C2 to C7, C3 to C8, C10 to C9, D2 to D1, D4 to D2, D1 to D3, D3 to D4, H3 to H1, H1 to H2, H2 to H3, J2 to J1, J6 to J2, J5 to J3, J1 to J5, J3 to J6, R6 to R1, R13 to R10, R4 to R11, R3 to R12, R9 to R13, R12 to R14, R8 to R15, R10 to R3, R7 to R4, R1 to R5, R11 to R6, R5 to R7, U2 to U1, U4 to U2, U5 to U3, U3 to U4
Connections:
- JP1 pad 2: VDD_STM -> Net-(JP1-C)
- R1 pad 2: VDD_STM -> Net-(JP1-C)
- R15 pad 2: VDD_STM -> Net-(JP2-C)
Routing:
- net VDD: track 0.00 -> 111.3 mm, vias 0 -> 3
- net /SCL: track 0.00 -> 77.9 mm, vias 0 -> 2
- net /SDA: track 0.00 -> 45.8 mm
- net VDD_STM: track 29.2 -> 0.00 mm
- net Net-(J4-CC2): track 15.9 -> 0.00 mm
- net Net-(JP1-C): track 0.00 -> 14.9 mm
- net Net-(JP2-C): track 0.00 -> 14.3 mm
- net Net-(J4-CC1): track 11.2 -> 0.00 mm
- net Net-(J7-CC2): track 0.00 -> 7.93 mm
- net Net-(J7-CC1): track 0.00 -> 7.80 mm
- net GND: track 32.2 -> 38.5 mm
- net V_USB: track 15.6 -> 20.8 mm
