File: STM32_sheild/_restore_backup_2026-07-19T20-16-48-722/STM32_sheild.kicad_sch (KiCad schematic)
At the start: 54 parts, among them J1 691210910002, J2 61612002121503, J3 691210910002, J4 629722010114, J5 CN10, J6 CN7, U1 DM-OLED096-636, U2 OPA333xxDBV, U3 OPA333xxDBV, U4 TPS63031DSK, U5 MCP73831-2-MC

Commit message: added footprint for oled + some other changes
Parts:
- renumbered C5 to C1, C8 to C10, C7 to C11, C4 to C2, C9 to C3, C11 to C4, C6 to C5, C1 to C6, C2 to C7, C3 to C8, C10 to C9, D2 to D1, D4 to D2, D1 to D3, D3 to D4, H3 to H1, H1 to H2, H2 to H3, J2 to J1, J6 to J2, J5 to J3, J1 to J5, J3 to J6, J4 to J7, JP1 to JP3, R6 to R1, R13 to R10, R4 to R11, R3 to R12, R9 to R13, R12 to R14, R8 to R15, R10 to R3, R7 to R4, R1 to R5, R11 to R6, R5 to R7, R14 to R8, R15 to R9, TP_GND1 to TP1, TP_3.3V_reg1 to TP2, TP_V_USB1 to TP3, TP_ADC1 to TP4, TP_ADC2 to TP5, TP5 to TP6, U2 to U1, U4 to U2, U5 to U3, U3 to U4, U1 to U5
