File: STM32_sheild/_restore_backup_2026-07-21T08-29-23-523/STM32_sheild.kicad_pcb (KiCad board)
At the start: 2 copper layers, 99 x 83.5 mm, 54 parts, among them J1 691210910002, J2 61612002121503, J3 691210910002, J4 629722010114, J5 CN10, J6 CN7, U1 DM-OLED096-636, U2 OPA333xxDBV, U3 OPA333xxDBV, U4 TPS63031DSK, U5 MCP73831-2-MC

Commit message: kicad crashed, hence copies
Other:
- board text removed: "ADC1"
- board text removed: "ADC2"
Changed lines of the file:
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@@
 		(tags "resistor")
 		(property "Reference" "R13"
-			(at 0 -1.5 0)
+			(at 3 0 0)
 			(layer "F.SilkS")
 			(effects
@@
 		)
 		(property "Value" "2k"
-			(at 2 0 90)
+			(at 2 -1 0)
 			(layer "F.Fab")
 			(effects
@@
 		(tags "WSON NoLead")
 		(property "Reference" "U4"
-			(at 0.5875 -1.9125 0)
+			(at 1.2875 -1.9125 0)
 			(layer "F.SilkS")
 			(effects
 				(font
-					(size 0.8 0.8)
+					(size 1 1)
 					(thickness 0.15)
 				)
@@
 		(tags "capacitor")
 		(property "Reference" "C10"
-			(at 3.1 1.2 180)
+			(at 2.5 1 180)
 			(layer "F.SilkS")
 			(effects
@@
 		(tags "Connector")
 		(property "Reference" "J3"
-			(at 1.94 -5.1 0)
+			(at 1.27 0 0)
 			(layer "F.SilkS")
 			(effects
@@
 		)
 		(fp_text user "${REFERENCE}"
-			(at -1.86 -5.1 0)
+			(at 1.27 0 0)
 			(layer "F.Fab")
 			(effects
@@
 		(tags "capacitor")
 		(property "Reference" "C6"
-			(at -2.8 0.1 0)
+			(at 0.5 1.5 0)
 			(layer "F.SilkS")
 			(effects
@@
 		(tags "Connector")
 		(property "Reference" "J1"
-			(at 4.2 5 0)
+			(at 1.27 0 0)
 			(layer "F.SilkS")
 			(effects
@@
 		)
 		(fp_text user "${REFERENCE}"
-			(at 4.2 5 0)
+			(at 1.27 0 0)
 			(layer "F.Fab")
 			(effects
@@
 		(tags "Connector")
 		(property "Reference" "J2"
-			(at -2.26 -5.66 0)
+			(at 0 0 0)
 			(layer "F.SilkS")
 			(effects
@@
 		)
 		(fp_text user "${REFERENCE}"
-			(at -2.26 -5.66 0)
+			(at 0 0 0)
 			(layer "F.Fab")
 			(effects
@@
 		(tags "capacitor")
 		(property "Reference" "C4"
-			(at 2.7 -0.9 270)
+			(at 2.4 0.7 270)
 			(layer "F.SilkS")
 			(effects
@@
 		(tags "capacitor")
 		(property "Reference" "C11"
-			(at 3 1.2 180)
+			(at 2.5 1 180)
 			(layer "F.SilkS")
 			(effects
@@
 		(tags "LED")
 		(property "Reference" "D4"
-			(at 0 1.6 0)
+			(at 0.9 -1.65 0)
 			(layer "F.SilkS")
 			(effects
@@
 		(tags "Through Hole Mount Test Points")
 		(property "Reference" "TP_3.3V_reg1"
-			(at -2 -2.7 180)
+			(at 0 -2.75 0)
 			(layer "F.SilkS")
 			(effects
 				(font
-					(size 0.8 0.8)
+					(size 1 1)
 					(thickness 0.15)
 				)
@@
 	)
 	(gr_text "Short and cut here \nto connect 3.3V reg"
-		(at 113.1 82.3 90)
-		(layer "F.SilkS")
-		(effects
-			(font
-				(size 0.8 0.8)
-				(thickness 0.15)
-			)
-			(justify left bottom)
-		)
-	)
-	(gr_text "ADC1"
-		(at 120.2 66.4 0)
+		(at 112.3 81.4 90)
 		(layer "F.SilkS")
 		(effects
 			(font
-				(size 1 1)
-				(thickness 0.15)
-			)
-			(justify left bottom)
-		)
-	)
-	(gr_text "ADC2"
-		(at 134.6 66.6 0)
-		(layer "F.SilkS")
-		(effects
-			(font
-				(size 1 1)
+				(size 0.75 0.75)
 				(thickness 0.15)
 			)
@@
 	)
 	(gr_text "Charger\nindicator\n"
-		(at 142.5 97 270)
+		(at 142.5 93.7 0)
 		(layer "F.SilkS")
 		(effects
@@
 	)
 	(segment
+		(start 160.8 103.9)
+		(end 160.9 103.8)
+		(width 0.25)
+		(layer "F.Cu")
+		(net "")
+	)
+	(segment
